File: hardware/tagger/tagger.sch (KiCad schematic (older format))
At the start: 7 parts

Commit message: Fix wrong pin in schematics
Parts:
- D?: symbol LED:APA102 -> tagger-rescue:APA102-LED
- D?: symbol LED:IR26-21C_L110_TR8 -> tagger-rescue:IR26-21C_L110_TR8-LED
- R?: symbol Device:R -> tagger-rescue:R-Device
- SW?: symbol Switch:SW_Push -> tagger-rescue:SW_Push-Switch
- U?: symbol RF_Module:ESP32-WROOM-32 -> tagger-rescue:ESP32-WROOM-32-RF_Module
- U?: symbol Driver_LED:WS2811 -> tagger-rescue:WS2811-Driver_LED
- U?: symbol Interface_Optical:TSOP312xx -> tagger-rescue:TSOP312xx-Interface_Optical
Connections:
- net at U?.12 (IO27): now also U?.3 (OUT)
- net at U?.27 (IO16): no longer U?.3 (OUT)
Other:
- moved on the sheet: D?, R?, SW?, U?
